File: KicadProject/SEAG/IO.kicad_sch (KiCad schematic)
At the start: 12 parts, among them J10 Screw_Terminal_01x02, J3 Screw_Terminal_01x02, J4 Screw_Terminal_01x02, J5 Screw_Terminal_01x02, J6 Screw_Terminal_01x02, J7 Screw_Terminal_01x02, J8 Screw_Terminal_01x02, J9 Screw_Terminal_01x02

Commit message: PCB rev 2
Parts:
- removed J10, J3, J4, J5, J6, J7, J8, J9: Screw_Terminal_01x02, TerminalBlock_Phoenix:TerminalBlock_Phoenix_MKDS-1,5-2_1x02_P5.00mm_Horizontal, symbol Connector:Screw_Terminal_01x02
- added C603, C604, C605, C606, C607, C608, C609, C610: 100n, Capacitor_SMD:C_0805_2012Metric, symbol Device:C
- added J14, J3: Screw_Terminal_01x08, SamacSys_Parts:1725711, symbol Connector:Screw_Terminal_01x08
- added J4, J5, J6, J7: Screw_Terminal_01x06, SamacSys_Parts:1725698, symbol Connector:Screw_Terminal_01x06
- added R601, R602, R603, R604, R605, R606, R607, R608: 10K, Resistor_SMD:R_0805_2012Metric, symbol Device:R
- renumbered C23 to C601, C24 to C602
Connections:
- net +3V3: now also R601.2, R602.2, R603.2, R604.2, R605.2, R606.2, R607.2, R608.2
- net GND: now also C603.2, C604.2, C605.2, C606.2, C607.2, C608.2, C609.2, C610.2, J4.3 (Pin_3), J4.6 (Pin_6), J5.3 (Pin_3), J5.6 (Pin_6), J6.3 (Pin_3), J6.6 (Pin_6), J7.3 (Pin_3), J7.6 (Pin_6)
- net Q0b: now also J14.1 (Pin_1)
- net Q0l: now also J3.1 (Pin_1)
- net Q1b: now also J14.2 (Pin_2)
- net Q1l: now also J3.2 (Pin_2)
- net Q2b: now also J14.3 (Pin_3)
- net Q2l: now also J3.3 (Pin_3)
- net Q3b: now also J14.4 (Pin_4)
- net Q3l: now also J3.4 (Pin_4)
- net Q4b: now also J14.5 (Pin_5)
- net Q4l: now also J3.5 (Pin_5)
- net Q5b: now also J14.6 (Pin_6)
- net Q5l: now also J3.6 (Pin_6)
- net Q6b: now also J14.7 (Pin_7)
- net Q6l: now also J3.7 (Pin_7)
- net Q7b: now also J14.8 (Pin_8)
- net Q7l: now also J3.8 (Pin_8)
- new net: J7.4 (Pin_4), R608.1
- new net: J7.1 (Pin_1), R607.1
- new net: J4.1 (Pin_1), R601.1
- new net: J6.4 (Pin_4), R606.1
- new net: J5.1 (Pin_1), R603.1
- new net: J5.4 (Pin_4), R604.1
- new net: J4.4 (Pin_4), R602.1
- new net: J6.1 (Pin_1), R605.1
- new net ToggleInput1: C603.1, J4.2 (Pin_2)
- new net ToggleInput2: C604.1, J4.5 (Pin_5)
- new net ToggleInput3: C605.1, J5.2 (Pin_2)
- new net ToggleInput4: C606.1, J5.5 (Pin_5)
- new net ToggleInput5: C607.1, J6.2 (Pin_2)
- new net ToggleInput6: C608.1, J6.5 (Pin_5)
- new net ToggleInput7: C609.1, J7.2 (Pin_2)
- new net ToggleInput8: C610.1, J7.5 (Pin_5)
Other:
- note added: "Toggle Input"
- moved on the sheet: C601, C602, U3, U4

Commit message: Added rotary encoder screw terminal
Parts:
- added J8: Screw_Terminal_01x03, SamacSys_Parts:2828343, symbol Connector:Screw_Terminal_01x03
- added R1: 10K, Resistor_SMD:R_0805_2012Metric, symbol Device:R
Connections:
- net +3V3: now also R1.2
- net GND: now also J8.1 (Pin_1)
- new net: J8.3 (Pin_3), R1.1
- new net PotInput: J8.2 (Pin_2)
Other:
- note added: "Potmeter Input"
Changed lines of the file:
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@@
+    (stroke (width 0) (type default))
+  )
+  (wire (pts (xy 50.165 74.295) (xy 50.165 77.47))
     (stroke (width 0) (type default))
   )
@@
     (stroke (width 0) (type default))
   )
+  (wire (pts (xy 37.465 74.295) (xy 50.165 74.295))
+    (stroke (width 0) (type default))
+  )
   (wire (pts (xy 202.565 52.705) (xy 207.645 52.705))
     (stroke (width 0) (type default))
@@
     (stroke (width 0) (type default))
   )
+  (wire (pts (xy 50.165 66.04) (xy 50.165 69.215))
+    (stroke (width 0) (type default))
+  )
   (wire (pts (xy 121.92 126.365) (xy 121.92 128.27))
     (stroke (width 0) (type default))
@@
     (stroke (width 0) (type default))
   )
+  (wire (pts (xy 37.465 69.215) (xy 40.64 69.215))
+    (stroke (width 0) (type default))
+  )
   (wire (pts (xy 202.565 40.005) (xy 207.645 40.005))
     (stroke (width 0) (type default))
@@
     (stroke (width 0) (type default))
   )
+  (wire (pts (xy 37.465 71.755) (xy 53.34 71.755))
+    (stroke (width 0) (type default))
+  )
   (wire (pts (xy 93.345 114.3) (xy 96.52 114.3))
     (stroke (width 0) (type default))
@@
   )
   (wire (pts (xy 111.125 103.505) (xy 111.125 106.68))
+    (stroke (width 0) (type default))
+  )
+  (wire (pts (xy 48.26 69.215) (xy 50.165 69.215))
     (stroke (width 0) (type default))
   )
@@
     (fill (type none))
   )
+  (rectangle (start 23.495 57.785) (end 66.04 86.36)
+    (stroke (width 0) (type dash))
+    (fill (type none))
+  )
   (rectangle (start 76.2 22.86) (end 147.955 177.8)
     (stroke (width 0) (type dash))
@@
   )
   (text "Decoupling" (at 23.495 22.225 0)
+    (effects (font (size 1.27 1.27)) (justify left bottom))
+  )
+  (text "Potmeter Input" (at 23.495 57.15 0)
     (effects (font (size 1.27 1.27)) (justify left bottom))
   )
@@
     )
   )
+  (global_label "PotInput" (shape input) (at 53.34 71.755 0) (fields_autoplaced)
+    (effects (font (size 1.27 1.27)) (justify left))
+    (property "Intersheetrefs" "${INTERSHEET_REFS}" (at 64.2474 71.755 0)
+      (effects (font (size 1.27 1.27)) (justify left) hide)
+    )
+  )
   (global_label "ShiftRegFClk" (shape input) (at 227.965 100.965 0) (fields_autoplaced)
     (effects (font (size 1.27 1.27)) (justify left))
@@
         (path "/37e7da6e-dab5-4e62-b28a-754ec4806405/b877551b-61ca-4466-b3f2-71fdb6767e79"
           (reference "#PWR035") (unit 1)
+        )
+      )
+    )
+  )
+  (symbol (lib_id "Device:R") (at 44.45 69.215 90) (unit 1)
+    (in_bom yes) (on_board yes) (dnp no)
+    (property "Reference" "R1" (at 44.45 65.405 90)
+      (effects (font (size 1.27 1.27)))
+    )
+    (property "Value" "10K" (at 44.45 67.31 90)
+      (effects (font (size 1.27 1.27)))
+    )
+    (property "Footprint" "Resistor_SMD:R_0805_2012Metric" (at 44.45 70.993 90)
+      (effects (font (size 1.27 1.27)) hide)
+    )
+    (property "Datasheet" "~" (at 44.45 69.215 0)
+      (effects (font (size 1.27 1.27)) hide)
+    )
+    (pin "1")
+    (pin "2")
+    (instances
+      (project "SEAG"
+        (path "/37e7da6e-dab5-4e62-b28a-754ec4806405/b877551b-61ca-4466-b3f2-71fdb6767e79"
+          (reference "R1") (unit 1)
+        )
+      )
+    )
+  )
+  (symbol (lib_id "Connector:Screw_Terminal_01x03") (at 32.385 71.755 180) (unit 1)
+    (in_bom yes) (on_board yes) (dnp no)
+    (property "Reference" "J8" (at 26.67 71.755 90)
+      (effects (font (size 1.27 1.27)))
+    )
+    (property "Value" "Screw_Terminal_01x03" (at 29.21 71.755 90)
+      (effects (font (size 1.27 1.27)))
+    )
+    (property "Footprint" "SamacSys_Parts:2828343" (at 32.385 71.755 0)
+      (effects (font (size 1.27 1.27)) hide)
+    )
+    (property "Datasheet" "~" (at 32.385 71.755 0)
+      (effects (font (size 1.27 1.27)) hide)
+    )
+    (pin "1")
+    (pin "2")
+    (pin "3")
+    (instances
+      (project "SEAG"
+        (path "/37e7da6e-dab5-4e62-b28a-754ec4806405/b877551b-61ca-4466-b3f2-71fdb6767e79"
+          (reference "J8") (unit 1)
         )
       )
@@
     )
   )
+  (symbol (lib_id "power:GND") (at 50.165 77.47 0) (unit 1)
+    (in_bom yes) (on_board yes) (dnp no) (fields_autoplaced)
+    (property "Reference" "#PWR078" (at 50.165 83.82 0)
+      (effects (font (size 1.27 1.27)) hide)
+    )
+    (property "Value" "GND" (at 50.165 81.915 0)
+      (effects (font (size 1.27 1.27)))
+    )
+    (property "Footprint" "" (at 50.165 77.47 0)
+      (effects (font (size 1.27 1.27)) hide)
+    )
+    (property "Datasheet" "" (at 50.165 77.47 0)
+      (effects (font (size 1.27 1.27)) hide)
+    )
+    (pin "1")
+    (instances
+      (project "SEAG"
+        (path "/37e7da6e-dab5-4e62-b28a-754ec4806405/b877551b-61ca-4466-b3f2-71fdb6767e79"
+          (reference "#PWR078") (unit 1)
+        )
+      )
+    )
+  )
   (symbol (lib_id "power:GND") (at 116.205 128.27 0) (unit 1)
     (in_bom yes) (on_board yes) (dnp no)
@@
         )
       )
+    )
+  )
+  (symbol (lib_id "power:+3V3") (at 50.165 66.04 0) (unit 1)
+    (in_bom yes) (on_board yes) (dnp no)
+    (property "Reference" "#PWR079" (at 50.165 69.85 0)
+      (effects (font (size 1.27 1.27)) hide)
+    )
+    (property "Value" "+3V3" (at 50.165 62.23 0)
+      (effects (font (size 1.27 1.27)))
+    )
+    (property "Footprint" "" (at 50.165 66.04 0)
+      (effects (font (size 1.27 1.27)) hide)
+    )
+    (property "Datasheet" "" (at 50.165 66.04 0)
+      (effects (font (size 1.27 1.27)) hide)
+    )
+    (pin "1")
+    (instances
+      (project "SEAG"
+        (path "/37e7da6e-dab5-4e62-b28a-754ec4806405/b877551b-61ca-4466-b3f2-71fdb6767e79"
+          (reference "#PWR079") (unit 1)
+        )
+      )

Commit message: Slight PCB changes
Parts:
- removed R1: 10K, Resistor_SMD:R_0805_2012Metric, symbol Device:R
Connections:
- net GND: no longer J8.1 (Pin_1)
- net RotEncoderIn1: now reaches J8.3 (Pin_3)
- net PotInput renamed RotEncoderIn2
- new net RotEncoderButton: J8.1 (Pin_1)
Changed lines of the file:
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@@
-    (stroke (width 0) (type default))
-  )
-  (wire (pts (xy 50.165 74.295) (xy 50.165 77.47))
     (stroke (width 0) (type default))
   )
@@
     (stroke (width 0) (type default))
   )
-  (wire (pts (xy 37.465 74.295) (xy 50.165 74.295))
+  (wire (pts (xy 37.465 74.295) (xy 41.91 74.295))
     (stroke (width 0) (type default))
   )
@@
     (stroke (width 0) (type default))
   )
-  (wire (pts (xy 50.165 66.04) (xy 50.165 69.215))
-    (stroke (width 0) (type default))
-  )
   (wire (pts (xy 121.92 126.365) (xy 121.92 128.27))
     (stroke (width 0) (type default))
@@
     (stroke (width 0) (type default))
   )
+  (wire (pts (xy 231.775 54.61) (xy 231.775 52.705))
+    (stroke (width 0) (type default))
+  )
   (wire (pts (xy 227.965 93.345) (xy 233.68 93.345))
     (stroke (width 0) (type default))
@@
     (stroke (width 0) (type default))
   )
-  (wire (pts (xy 227.965 50.165) (xy 238.76 50.165))
+  (wire (pts (xy 227.965 50.165) (xy 236.855 50.165))
     (stroke (width 0) (type default))
   )
@@
     (stroke (width 0) (type default))
   )
-  (wire (pts (xy 37.465 69.215) (xy 40.64 69.215))
+  (wire (pts (xy 37.465 69.215) (xy 41.91 69.215))
     (stroke (width 0) (type default))
   )
@@
     (stroke (width 0) (type default))
   )
+  (wire (pts (xy 231.14 106.045) (xy 227.965 106.045))
+    (stroke (width 0) (type default))
+  )
   (wire (pts (xy 93.345 71.12) (xy 96.52 71.12))
     (stroke (width 0) (type default))
@@
     (stroke (width 0) (type default))
   )
-  (wire (pts (xy 37.465 71.755) (xy 53.34 71.755))
+  (wire (pts (xy 37.465 71.755) (xy 41.91 71.755))
     (stroke (width 0) (type default))
   )
@@
     (stroke (width 0) (type default))
   )
-  (wire (pts (xy 227.965 52.705) (xy 234.315 52.705))
+  (wire (pts (xy 231.775 54.61) (xy 236.22 54.61))
     (stroke (width 0) (type default))
   )
@@
     (stroke (width 0) (type default))
   )
+  (wire (pts (xy 231.775 52.705) (xy 227.965 52.705))
+    (stroke (width 0) (type default))
+  )
   (wire (pts (xy 106.045 83.82) (xy 106.045 92.71))
     (stroke (width 0) (type default))
@@
     (stroke (width 0) (type default))
   )
-  (wire (pts (xy 48.26 69.215) (xy 50.165 69.215))
-    (stroke (width 0) (type default))
-  )
   (wire (pts (xy 202.565 45.085) (xy 207.645 45.085))
     (stroke (width 0) (type default))
@@
     (stroke (width 0) (type default))
   )
-  (wire (pts (xy 227.965 106.045) (xy 234.315 106.045))
+  (wire (pts (xy 231.14 107.315) (xy 231.14 106.045))
+    (stroke (width 0) (type default))
+  )
+  (wire (pts (xy 231.14 107.315) (xy 234.95 107.315))
     (stroke (width 0) (type default))
   )
@@
   (label "Q4b" (at 202.565 47.625 0) (fields_autoplaced)
     (effects (font (size 1.27 1.27)) (justify left bottom))
+  )
+  (global_label "RotEncoderButton" (shape input) (at 41.91 74.295 0) (fields_autoplaced)
+    (effects (font (size 1.27 1.27)) (justify left))
+    (property "Intersheetrefs" "${INTERSHEET_REFS}" (at 61.7677 74.295 0)
+      (effects (font (size 1.27 1.27)) (justify left) hide)
+    )
+  )
+  (global_label "RotEncoderIn1" (shape input) (at 41.91 69.215 0) (fields_autoplaced)
+    (effects (font (size 1.27 1.27)) (justify left))
+    (property "Intersheetrefs" "${INTERSHEET_REFS}" (at 58.5626 69.215 0)
+      (effects (font (size 1.27 1.27)) (justify left) hide)
+    )
   )
   (global_label "ToggleInput7" (shape input) (at 126.365 148.59 0) (fields_autoplaced)
@@
     )
   )
-  (global_label "PotInput" (shape input) (at 53.34 71.755 0) (fields_autoplaced)
+  (global_label "RotEncoderIn2" (shape input) (at 41.91 71.755 0) (fields_autoplaced)
     (effects (font (size 1.27 1.27)) (justify left))
-    (property "Intersheetrefs" "${INTERSHEET_REFS}" (at 64.2474 71.755 0)
+    (property "Intersheetrefs" "${INTERSHEET_REFS}" (at 58.5626 71.755 0)
       (effects (font (size 1.27 1.27)) (justify left) hide)
     )
@@
     )
   )
-  (global_label "ShiftRegBarStoClk" (shape input) (at 238.76 50.165 0) (fields_autoplaced)
+  (global_label "ShiftRegBarStoClk" (shape input) (at 236.855 50.165 0) (fields_autoplaced)
     (effects (font (size 1.27 1.27)) (justify left))
-    (property "Intersheetrefs" "${INTERSHEET_REFS}" (at 258.9202 50.165 0)
+    (property "Intersheetrefs" "${INTERSHEET_REFS}" (at 257.0152 50.165 0)
       (effects (font (size 1.27 1.27)) (justify left) hide)
     )
@@
         (path "/37e7da6e-dab5-4e62-b28a-754ec4806405/b877551b-61ca-4466-b3f2-71fdb6767e79"
           (reference "#PWR035") (unit 1)
-        )
-      )
-    )
-  )
-  (symbol (lib_id "Device:R") (at 44.45 69.215 90) (unit 1)
-    (in_bom yes) (on_board yes) (dnp no)
-    (property "Reference" "R1" (at 44.45 65.405 90)
-      (effects (font (size 1.27 1.27)))
-    )
-    (property "Value" "10K" (at 44.45 67.31 90)
-      (effects (font (size 1.27 1.27)))
-    )
-    (property "Footprint" "Resistor_SMD:R_0805_2012Metric" (at 44.45 70.993 90)
-      (effects (font (size 1.27 1.27)) hide)
-    )
-    (property "Datasheet" "~" (at 44.45 69.215 0)
-      (effects (font (size 1.27 1.27)) hide)
-    )
-    (pin "1")
-    (pin "2")
-    (instances
-      (project "SEAG"
-        (path "/37e7da6e-dab5-4e62-b28a-754ec4806405/b877551b-61ca-4466-b3f2-71fdb6767e79"
-          (reference "R1") (unit 1)
         )
       )
@@
     )
   )
-  (symbol (lib_id "power:GND") (at 50.165 77.47 0) (unit 1)
-    (in_bom yes) (on_board yes) (dnp no) (fields_autoplaced)
-    (property "Reference" "#PWR078" (at 50.165 83.82 0)
-      (effects (font (size 1.27 1.27)) hide)
-    )
-    (property "Value" "GND" (at 50.165 81.915 0)
-      (effects (font (size 1.27 1.27)))
-    )
-    (property "Footprint" "" (at 50.165 77.47 0)
-      (effects (font (size 1.27 1.27)) hide)
-    )
-    (property "Datasheet" "" (at 50.165 77.47 0)
-      (effects (font (size 1.27 1.27)) hide)
-    )
-    (pin "1")
-    (instances
-      (project "SEAG"
-        (path "/37e7da6e-dab5-4e62-b28a-754ec4806405/b877551b-61ca-4466-b3f2-71fdb6767e79"
-          (reference "#PWR078") (unit 1)
-        )
-      )
-    )
-  )
   (symbol (lib_id "power:GND") (at 116.205 128.27 0) (unit 1)
     (in_bom yes) (on_board yes) (dnp no)
@@
     )
   )
-  (symbol (lib_id "power:+3V3") (at 234.315 52.705 0) (unit 1)
+  (symbol (lib_id "power:+3V3") (at 236.22 54.61 0) (unit 1)
     (in_bom yes) (on_board yes) (dnp no) (fields_autoplaced)
-    (property "Reference" "#PWR043" (at 234.315 56.515 0)
-      (effects (font (size 1.27 1.27)) hide)
-    )
-    (property "Value" "+3V3" (at 234.315 47.625 0)
-      (effects (font (size 1.27 1.27)) hide)
-    )
-    (property "Footprint" "" (at 234.315 52.705 0)
-      (effects (font (size 1.27 1.27)) hide)
-    )
-    (property "Datasheet" "" (at 234.315 52.705 0)
+    (property "Reference" "#PWR043" (at 236.22 58.42 0)
+      (effects (font (size 1.27 1.27)) hide)
+    )
+    (property "Value" "+3V3" (at 236.22 49.53 0)
+      (effects (font (size 1.27 1.27)) hide)
+    )
+    (property "Footprint" "" (at 236.22 54.61 0)
+      (effects (font (size 1.27 1.27)) hide)
+    )
+    (property "Datasheet" "" (at 236.22 54.61 0)
       (effects (font (size 1.27 1.27)) hide)
     )
@@
   )
   (symbol (lib_id "power:GND") (at 259.715 46.99 0) (unit 1)
-    (in_bom yes) (on_board yes) (dnp no) (fields_autoplaced)
+    (in_bom yes) (on_board yes) (dnp no)
     (property "Reference" "#PWR042" (at 259.715 53.34 0)
       (effects (font (size 1.27 1.27)) hide)
@@
     )
   )
-  (symbol (lib_id "power:+3V3") (at 234.315 106.045 0) (unit 1)
+  (symbol (lib_id "power:+3V3") (at 234.95 107.315 0) (unit 1)
     (in_bom yes) (on_board yes) (dnp no) (fields_autoplaced)
-    (property "Reference" "#PWR046" (at 234.315 109.855 0)
-      (effects (font (size 1.27 1.27)) hide)
-    )
-    (property "Value" "+3V3" (at 234.315 100.965 0)
-      (effects (font (size 1.27 1.27)) hide)
-    )
-    (property "Footprint" "" (at 234.315 106.045 0)
-      (effects (font (size 1.27 1.27)) hide)
-    )
-    (property "Datasheet" "" (at 234.315 106.045 0)
+    (property "Reference" "#PWR046" (at 234.95 111.125 0)
+      (effects (font (size 1.27 1.27)) hide)
+    )
+    (property "Value" "+3V3" (at 234.95 102.235 0)
+      (effects (font (size 1.27 1.27)) hide)
+    )
+    (property "Footprint" "" (at 234.95 107.315 0)
+      (effects (font (size 1.27 1.27)) hide)
+    )
+    (property "Datasheet" "" (at 234.95 107.315 0)
       (effects (font (size 1.27 1.27)) hide)
     )
@@
         )
       )
-    )
-  )
-  (symbol (lib_id "power:+3V3") (at 50.165 66.04 0) (unit 1)
-    (in_bom yes) (on_board yes) (dnp no)
-    (property "Reference" "#PWR079" (at 50.165 69.85 0)
-      (effects (font (size 1.27 1.27)) hide)
-    )
-    (property "Value" "+3V3" (at 50.165 62.23 0)
-      (effects (font (size 1.27 1.27)))
-    )
-    (property "Footprint" "" (at 50.165 66.04 0)
-      (effects (font (size 1.27 1.27)) hide)
-    )
-    (property "Datasheet" "" (at 50.165 66.04 0)
-      (effects (font (size 1.27 1.27)) hide)
-    )
-    (pin "1")
-    (instances
-      (project "SEAG"
-        (path "/37e7da6e-dab5-4e62-b28a-754ec4806405/b877551b-61ca-4466-b3f2-71fdb6767e79"
-          (reference "#PWR079") (unit 1)
-        )
-      )
