File: KicadProject/SEAG/IO.kicad_sch (KiCad schematic)
At the start: 27 parts, among them J14 Screw_Terminal_01x08, J3 Screw_Terminal_01x08, J4 Screw_Terminal_01x06, J5 Screw_Terminal_01x06, J6 Screw_Terminal_01x06, J7 Screw_Terminal_01x06, J8 Screw_Terminal_01x03

Commit message: Added header
Parts:
- added R609: 10K, Resistor_SMD:R_0805_2012Metric, symbol Device:R
Connections:
- net +3V3: now also R609.1
- net RotEncoderButton: now also R609.2
Other:
- moved on the sheet: J8
Changed lines of the file:
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@@
   (junction (at 38.735 40.64) (diameter 0) (color 0 0 0 0)
+  )
+  (junction (at 39.37 78.105) (diameter 0) (color 0 0 0 0)
   )
   (junction (at 121.92 43.18) (diameter 0) (color 0 0 0 0)
@@
     (stroke (width 0) (type default))
   )
-  (wire (pts (xy 37.465 74.295) (xy 41.91 74.295))
+  (wire (pts (xy 37.465 78.105) (xy 39.37 78.105))
     (stroke (width 0) (type default))
   )
@@
     (stroke (width 0) (type default))
   )
-  (wire (pts (xy 37.465 69.215) (xy 41.91 69.215))
+  (wire (pts (xy 37.465 73.025) (xy 41.91 73.025))
     (stroke (width 0) (type default))
   )
@@
     (stroke (width 0) (type default))
   )
-  (wire (pts (xy 37.465 71.755) (xy 41.91 71.755))
+  (wire (pts (xy 37.465 75.565) (xy 41.91 75.565))
     (stroke (width 0) (type default))
   )
@@
     (stroke (width 0) (type default))
   )
+  (wire (pts (xy 39.37 63.5) (xy 39.37 62.23))
+    (stroke (width 0) (type default))
+  )
   (wire (pts (xy 104.14 114.3) (xy 106.045 114.3))
     (stroke (width 0) (type default))
@@
     (stroke (width 0) (type default))
   )
+  (wire (pts (xy 39.37 71.12) (xy 39.37 78.105))
+    (stroke (width 0) (type default))
+  )
   (wire (pts (xy 111.125 76.2) (xy 111.125 92.71))
     (stroke (width 0) (type default))
@@
   )
   (wire (pts (xy 202.565 55.245) (xy 207.645 55.245))
+    (stroke (width 0) (type default))
+  )
+  (wire (pts (xy 39.37 78.105) (xy 41.91 78.105))
     (stroke (width 0) (type default))
   )
@@
     (fill (type none))
   )
-  (rectangle (start 23.495 57.785) (end 66.04 86.36)
+  (rectangle (start 23.495 55.88) (end 66.04 86.36)
     (stroke (width 0) (type dash))
     (fill (type none))
@@
     (effects (font (size 1.27 1.27)) (justify left bottom))
   )
-  (text "Potmeter Input" (at 23.495 57.15 0)
+  (text "Potmeter Input" (at 23.495 55.88 0)
     (effects (font (size 1.27 1.27)) (justify left bottom))
   )
@@
     (effects (font (size 1.27 1.27)) (justify right bottom))
   )
-  (label "~{OE}b" (at 259.715 98.425 180) (fields_autoplaced)
-    (effects (font (size 1.27 1.27)) (justify right bottom))
-  )
   (label "Q2l" (at 200.66 95.885 180) (fields_autoplaced)
     (effects (font (size 1.27 1.27)) (justify right bottom))
@@
     (effects (font (size 1.27 1.27)) (justify right bottom))
   )
-  (label "~{OE}b" (at 259.715 45.085 180) (fields_autoplaced)
-    (effects (font (size 1.27 1.27)) (justify right bottom))
-  )
   (label "Q3b" (at 202.565 45.085 0) (fields_autoplaced)
     (effects (font (size 1.27 1.27)) (justify left bottom))
@@
     (effects (font (size 1.27 1.27)) (justify left bottom))
   )
-  (global_label "RotEncoderButton" (shape input) (at 41.91 74.295 0) (fields_autoplaced)
+  (global_label "RotEncoderButton" (shape input) (at 41.91 78.105 0) (fields_autoplaced)
     (effects (font (size 1.27 1.27)) (justify left))
-    (property "Intersheetrefs" "${INTERSHEET_REFS}" (at 61.7677 74.295 0)
+    (property "Intersheetrefs" "${INTERSHEET_REFS}" (at 61.7677 78.105 0)
       (effects (font (size 1.27 1.27)) (justify left) hide)
     )
   )
-  (global_label "RotEncoderIn1" (shape input) (at 41.91 69.215 0) (fields_autoplaced)
+  (global_label "RotEncoderIn1" (shape input) (at 41.91 73.025 0) (fields_autoplaced)
     (effects (font (size 1.27 1.27)) (justify left))
-    (property "Intersheetrefs" "${INTERSHEET_REFS}" (at 58.5626 69.215 0)
+    (property "Intersheetrefs" "${INTERSHEET_REFS}" (at 58.5626 73.025 0)
       (effects (font (size 1.27 1.27)) (justify left) hide)
     )
@@
     )
   )
-  (global_label "RotEncoderIn2" (shape input) (at 41.91 71.755 0) (fields_autoplaced)
+  (global_label "RotEncoderIn2" (shape input) (at 41.91 75.565 0) (fields_autoplaced)
     (effects (font (size 1.27 1.27)) (justify left))
-    (property "Intersheetrefs" "${INTERSHEET_REFS}" (at 58.5626 71.755 0)
+    (property "Intersheetrefs" "${INTERSHEET_REFS}" (at 58.5626 75.565 0)
       (effects (font (size 1.27 1.27)) (justify left) hide)
     )
@@
     )
   )
-  (symbol (lib_id "Connector:Screw_Terminal_01x03") (at 32.385 71.755 180) (unit 1)
-    (in_bom yes) (on_board yes) (dnp no)
-    (property "Reference" "J8" (at 26.67 71.755 90)
-      (effects (font (size 1.27 1.27)))
-    )
-    (property "Value" "Screw_Terminal_01x03" (at 29.21 71.755 90)
-      (effects (font (size 1.27 1.27)))
-    )
-    (property "Footprint" "SamacSys_Parts:2828343" (at 32.385 71.755 0)
-      (effects (font (size 1.27 1.27)) hide)
-    )
-    (property "Datasheet" "~" (at 32.385 71.755 0)
+  (symbol (lib_id "Connector:Screw_Terminal_01x03") (at 32.385 75.565 180) (unit 1)
+    (in_bom yes) (on_board yes) (dnp no)
+    (property "Reference" "J8" (at 26.67 75.565 90)
+      (effects (font (size 1.27 1.27)))
+    )
+    (property "Value" "Screw_Terminal_01x03" (at 29.21 75.565 90)
+      (effects (font (size 1.27 1.27)))
+    )
+    (property "Footprint" "SamacSys_Parts:2828343" (at 32.385 75.565 0)
+      (effects (font (size 1.27 1.27)) hide)
+    )
+    (property "Datasheet" "~" (at 32.385 75.565 0)
       (effects (font (size 1.27 1.27)) hide)
     )
@@
     )
   )
+  (symbol (lib_id "Device:R") (at 39.37 67.31 0) (unit 1)
+    (in_bom yes) (on_board yes) (dnp no) (fields_autoplaced)
+    (property "Reference" "R609" (at 41.91 66.04 0)
+      (effects (font (size 1.27 1.27)) (justify left))
+    )
+    (property "Value" "10K" (at 41.91 68.58 0)
+      (effects (font (size 1.27 1.27)) (justify left))
+    )
+    (property "Footprint" "Resistor_SMD:R_0805_2012Metric" (at 37.592 67.31 90)
+      (effects (font (size 1.27 1.27)) hide)
+    )
+    (property "Datasheet" "~" (at 39.37 67.31 0)
+      (effects (font (size 1.27 1.27)) hide)
+    )
+    (pin "2")
+    (pin "1")
+    (instances
+      (project "SEAG"
+        (path "/37e7da6e-dab5-4e62-b28a-754ec4806405/b877551b-61ca-4466-b3f2-71fdb6767e79"
+          (reference "R609") (unit 1)
+        )
+      )
+    )
+  )
   (symbol (lib_id "Connector:Screw_Terminal_01x08") (at 191.77 45.085 0) (mirror y) (unit 1)
     (in_bom yes) (on_board yes) (dnp no)
@@
         )
       )
+    )
+  )
+  (symbol (lib_id "power:+3V3") (at 39.37 62.23 0) (unit 1)
+    (in_bom yes) (on_board yes) (dnp no) (fields_autoplaced)
+    (property "Reference" "#PWR078" (at 39.37 66.04 0)
+      (effects (font (size 1.27 1.27)) hide)
+    )
+    (property "Value" "+3V3" (at 39.37 57.785 0)
+      (effects (font (size 1.27 1.27)))
+    )
+    (property "Footprint" "" (at 39.37 62.23 0)
+      (effects (font (size 1.27 1.27)) hide)
+    )
+    (property "Datasheet" "" (at 39.37 62.23 0)
+      (effects (font (size 1.27 1.27)) hide)
+    )
+    (pin "1")
+    (instances
+      (project "SEAG"
+        (path "/37e7da6e-dab5-4e62-b28a-754ec4806405/b877551b-61ca-4466-b3f2-71fdb6767e79"
+          (reference "#PWR078") (unit 1)
+        )
+      )
